File: ARII/ActionReplayAmiga/ActionReplayAmiga.kicad_pcb (KiCad board)
At the start: 2 copper layers, 0 parts

Commit message: Started U2 and added board edge cuts 96x114mm Indents are 10.1mm deep and 2.8mm heigh
Other:
- board outline added: 114 x 96 mm
Changed lines of the file:
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@@
   (general
     (thickness 1.6)
-    (drawings 0)
+    (drawings 12)
     (tracks 0)
     (zones 0)
@@
     (solder_mask_min_width 0.25)
     (aux_axis_origin 0 0)
-    (visible_elements FFFFFF7F)
+    (visible_elements 7FFFFFFF)
     (pcbplotparams
       (layerselection 0x010fc_ffffffff)
@@
     (uvia_drill 0.1)
   )
+  (gr_line (start 134 88.1) (end 134 20) (layer Edge.Cuts) (width 0.1))
+  (gr_line (start 20 88.1) (end 20 20) (layer Edge.Cuts) (width 0.1))
+  (gr_line (start 134 116) (end 134 90.9) (layer Edge.Cuts) (width 0.1))
+  (gr_line (start 20 116) (end 20 90.9) (layer Edge.Cuts) (width 0.1))
+  (gr_line (start 30.3 88.1) (end 20 88.1) (layer Edge.Cuts) (width 0.1))
+  (gr_line (start 30.3 90.9) (end 30.3 88.1) (layer Edge.Cuts) (width 0.1))
+  (gr_line (start 20 90.9) (end 30.3 90.9) (layer Edge.Cuts) (width 0.1))
+  (gr_line (start 123.7 88.1) (end 134 88.1) (layer Edge.Cuts) (width 0.1))
+  (gr_line (start 123.7 90.9) (end 123.7 88.1) (layer Edge.Cuts) (width 0.1))
+  (gr_line (start 134 90.9) (end 123.7 90.9) (layer Edge.Cuts) (width 0.1))
+  (gr_line (start 134 116) (end 20 116) (layer Edge.Cuts) (width 0.1))
+  (gr_line (start 20 20) (end 134 20) (layer Edge.Cuts) (width 0.1))
 )
