File: ARIII/kicad/AR3.kicad_sch (KiCad schematic)
At the start: 30 parts, among them U1-WHITE PAL16L8, U2-RED PAL16L8, U3-BROWN PAL16L8, U4-GREEN PAL16L8, U5-BLUE PAL16L8

Commit message: Update AR3 - update project to KiCad 7 - add missing ROM connections - add annotated picture - rename ROMs according to picture
Parts:
- gave numbers to parts that had none: 2
Connections:
- net D0: now also U6.13 (O0)
- net D1: now also U6.14 (O1)
- net D2: now also U6.15 (O2)
- net D3: now also U6.17 (O3)
- net D4: now also U6.18 (O4)
- net D5: now also U6.19 (O5)
- net D6: now also U6.20 (O6)
- net D7: now also U6.21 (O7)
